File: Plakat.sch (EAGLE design)
At the start: 25 parts, among them X1 USB-MICROB

Commit message: Nothing
Parts:
- C3: device resistor:CPOL-EUD/7343-31W -> rcl:CPOL-EU
Changed lines of the file:
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@@
 <part name="C1" library="rcl" deviceset="C-EU" device="C0805" value="10uF"/>
 <part name="D2" library="diode" deviceset="1N581*" device="" technology="9-T"/>
-<part name="C3" library="resistor" deviceset="CPOL-EU" device="D/7343-31W" value="1uF"/>
 <part name="C4" library="rcl" deviceset="C-EU" device="C0805" value="100nF"/>
 <part name="GND1" library="supply1" deviceset="GND" device=""/>
@@
 <part name="GND8" library="supply1" deviceset="GND" device=""/>
 <part name="L1" library="BOURNS" deviceset="SRD0604-101KL" device="" value="100uH"/>
+<part name="C3" library="rcl" deviceset="CPOL-EU" device="" value="1uF"/>
 </parts>
 <sheets>
@@
 <attribute name="NAME" x="-95.123" y="69.596" size="1.778" layer="95" rot="MR90"/>
 </instance>
-<instance part="C3" gate="G$1" x="-55.88" y="71.12"/>
 <instance part="C4" gate="G$1" x="-48.26" y="71.12"/>
 <instance part="GND1" gate="1" x="-55.88" y="58.42" rot="MR0"/>
@@
 <instance part="GND8" gate="1" x="-33.02" y="-116.84" rot="R180"/>
 <instance part="L1" gate="G$1" x="-81.28" y="76.2" rot="MR0"/>
+<instance part="C3" gate="G$1" x="-55.88" y="71.12"/>
 </instances>
 <busses>
@@
 <pinref part="C4" gate="G$1" pin="2"/>
 <wire x1="-48.26" y1="66.04" x2="-48.26" y2="63.5" width="0.1524" layer="91"/>
-<pinref part="C3" gate="G$1" pin="-"/>
 <wire x1="-48.26" y1="63.5" x2="-55.88" y2="63.5" width="0.1524" layer="91"/>
 <wire x1="-55.88" y1="63.5" x2="-55.88" y2="66.04" width="0.1524" layer="91"/>
@@
 <wire x1="-55.88" y1="63.5" x2="-55.88" y2="60.96" width="0.1524" layer="91"/>
 <junction x="-55.88" y="63.5"/>
+<pinref part="C3" gate="G$1" pin="-"/>
 </segment>
 <segment>
@@
 <wire x1="-30.48" y1="76.2" x2="-48.26" y2="76.2" width="0.1524" layer="91"/>
 <wire x1="-48.26" y1="76.2" x2="-48.26" y2="73.66" width="0.1524" layer="91"/>
-<pinref part="C3" gate="G$1" pin="+"/>
 <wire x1="-48.26" y1="76.2" x2="-55.88" y2="76.2" width="0.1524" layer="91"/>
 <wire x1="-55.88" y1="76.2" x2="-55.88" y2="73.66" width="0.1524" layer="91"/>
@@
 <junction x="-43.18" y="53.34"/>
 <pinref part="L1" gate="G$1" pin="1"/>
-</segment>
-<segment>
+<pinref part="C3" gate="G$1" pin="+"/>
+</segment>
+<segment>
