File: Plakat_залипуха.brd (EAGLE design)
At the start: 82.4 x 68.1 mm, 25 parts, among them X1 USB-MICROB

Commit message: Edited plakat_залипуха
Parts:
- renumbered D2 to D1, LED1 to VD1
Routing:
- net N$1: track 24.1 -> 22.1 mm
Changed lines of the file:
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@@
 </autorouter>
 <elements>
-<element name="LED1" library="eagle-ltspice" package="LED_1206" value="" x="118" y="62.02" smashed="yes">
+<element name="VD1" library="eagle-ltspice" package="LED_1206" value="" x="118" y="62.02" smashed="yes">
 <attribute name="SPICETYPE" value="diode" x="118" y="62.02" size="1.778" layer="27" display="off"/>
 <attribute name="SPICEMODEL" value="NONE" x="118" y="62.02" size="1.778" layer="27" display="off"/>
@@
 <attribute name="VALUE" x="67.52" y="65.08" size="0.6096" layer="27"/>
 </element>
-<element name="D2" library="diode" package="DO41-7.6" value="1N5819-T" x="113.15" y="40.68" rot="R180"/>
+<element name="D1" library="diode" package="DO41-7.6" value="1N5819-T" x="113.15" y="40.68" rot="R180"/>
 <element name="DA1" library="LM2594" package="LM2495" value="LM2594" x="115.02" y="51.15" rot="R180"/>
 <element name="R1" library="eagle-ltspice" package="R0805" value="470" x="117.99" y="64.48" smashed="yes" rot="R180">
@@
 <signal name="GND">
 <contactref element="C1" pad="2"/>
-<contactref element="D2" pad="A"/>
+<contactref element="D1" pad="A"/>
 <contactref element="C2" pad="2"/>
 <contactref element="DA1" pad="ON/OFF"/>
 <contactref element="DA1" pad="GND"/>
-<contactref element="LED1" pad="C"/>
+<contactref element="VD1" pad="C"/>
 <contactref element="C4" pad="2"/>
 <contactref element="C5" pad="2"/>
@@
 </signal>
 <signal name="N$2">
-<contactref element="D2" pad="C"/>
+<contactref element="D1" pad="C"/>
 <contactref element="L1" pad="2"/>
 <wire x1="116.925" y1="40.715" x2="116.96" y2="40.68" width="0.3048" layer="1"/>
@@
 <contactref element="DA1" pad="V(IN)"/>
 <contactref element="C1" pad="1"/>
-<contactref element="R1" pad="2"/>
 <wire x1="112.51" y1="68.09" x2="113" y2="67.6" width="0.3048" layer="1"/>
 <wire x1="113" y1="67.6" x2="114.38" y2="67.6" width="0.3048" layer="1"/>
@@
 <wire x1="114.46" y1="65.29" x2="114.46" y2="67.52" width="0.3048" layer="1"/>
 <wire x1="114.46" y1="67.52" x2="114.44" y2="67.54" width="0.3048" layer="1"/>
-<wire x1="117.04" y1="64.48" x2="115.02" y2="64.48" width="0.3048" layer="1"/>
 <wire x1="115.02" y1="64.48" x2="115" y2="64.5" width="0.3048" layer="1"/>
 <contactref element="X1" pad="D+"/>
+<contactref element="R1" pad="2"/>
 <wire x1="112.51" y1="68.09" x2="111.21" y2="71.84" width="0" layer="19" extent="1-1"/>
+<wire x1="117.04" y1="64.48" x2="115.02" y2="64.48" width="0" layer="19" extent="1-1"/>
 </signal>
 <signal name="N$4">
 <contactref element="R1" pad="1"/>
-<contactref element="LED1" pad="A"/>
+<contactref element="VD1" pad="A"/>
 <wire x1="116.96" y1="62.402" x2="116.578" y2="62.02" width="0.3048" layer="1"/>
 <wire x1="118.94" y1="64.48" x2="118.94" y2="64.04" width="0.3048" layer="1"/>
@@
 <wire x1="85.5" y1="50.7" x2="85.5" y2="49.43" width="0.3048" layer="1"/>
 <wire x1="85.5" y1="49.43" x2="85.49" y2="49.42" width="0.3048" layer="1"/>
+<contactref element="X3" pad="1"/>
+<wire x1="93.14" y1="63.24" x2="93.4" y2="63.5" width="0.3048" layer="1"/>
+<wire x1="93.4" y1="63.5" x2="95.7" y2="63.5" width="0.3048" layer="1"/>
+<wire x1="95.7" y1="63.5" x2="96.7" y2="64.5" width="0.3048" layer="1"/>
+<wire x1="96.7" y1="64.5" x2="96.7" y2="66.6" width="0.3048" layer="1"/>
+<wire x1="96.7" y1="66.6" x2="96.67" y2="66.63" width="0.3048" layer="1"/>
 <contactref element="C2" pad="1"/>
 <contactref element="DA1" pad="FB"/>
@@
 <wire x1="68.6" y1="52.1" x2="68.6" y2="53.395" width="0.3048" layer="1"/>
 <wire x1="68.6" y1="53.395" x2="68.605" y2="53.4" width="0.3048" layer="1"/>
-<contactref element="X3" pad="1"/>
-<wire x1="93.14" y1="63.24" x2="93.4" y2="63.5" width="0.3048" layer="1"/>
-<wire x1="93.4" y1="63.5" x2="95.7" y2="63.5" width="0.3048" layer="1"/>
-<wire x1="95.7" y1="63.5" x2="96.7" y2="64.5" width="0.3048" layer="1"/>
-<wire x1="96.7" y1="64.5" x2="96.7" y2="66.6" width="0.3048" layer="1"/>
-<wire x1="96.7" y1="66.6" x2="96.67" y2="66.63" width="0.3048" layer="1"/>
 <wire x1="93.14" y1="61.66" x2="93.14" y2="63.24" width="0" layer="19" extent="1-1"/>
 <wire x1="85.3134" y1="50.8866" x2="85.2234" y2="60.9234" width="0" layer="19" extent="1-1"/>
