File: EAGLE/Analog/Analog_1.brd (EAGLE design)
At the start: 297 x 210 mm, 7 parts

Commit message: Я уже ничего не помню
Other:
- board size 297 x 210 mm -> 297 x 200 mm
Changed lines of the file:
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@@
 <?xml version="1.0" encoding="utf-8"?>
 <!DOCTYPE eagle SYSTEM "eagle.dtd">
-<eagle version="7.5.0">
+<eagle version="8.2.1">
 <drawing>
 <settings>
@@
 <board>
 <plain>
-<wire x1="0" y1="210" x2="0" y2="0" width="0.4064" layer="20"/>
+<wire x1="0" y1="200" x2="0" y2="0" width="0.4064" layer="20"/>
 <wire x1="0" y1="0" x2="254" y2="0" width="0.4064" layer="20"/>
-<wire x1="297" y1="28" x2="297" y2="210" width="0.4064" layer="20"/>
-<wire x1="297" y1="210" x2="0" y2="210" width="0.4064" layer="20"/>
+<wire x1="297" y1="28" x2="297" y2="200" width="0.4064" layer="20"/>
+<wire x1="297" y1="200" x2="0" y2="200" width="0.4064" layer="20"/>
 <wire x1="254" y1="28" x2="297" y2="28" width="0.4064" layer="20"/>
 <wire x1="254" y1="28" x2="254" y2="0" width="0.4064" layer="20"/>
-<text x="5" y="200" size="6.4516" layer="1">1</text>
+<text x="5" y="190" size="6.4516" layer="1">1</text>
 <hole x="4" y="4" drill="3"/>
-<hole x="4" y="206" drill="3"/>
-<hole x="294" y="206" drill="3"/>
+<hole x="4" y="196" drill="3"/>
+<hole x="294" y="196" drill="3"/>
 <hole x="294" y="31" drill="3"/>
 <hole x="250" y="4" drill="3"/>
 <hole x="4" y="105" drill="3"/>
 <hole x="294" y="105" drill="3"/>
-<hole x="148.5" y="206" drill="3"/>
+<hole x="148.5" y="196" drill="3"/>
 <hole x="148.5" y="4" drill="3"/>
 <hole x="148.5" y="105" drill="3"/>
@@
 <vertex x="254" y="28"/>
 <vertex x="297" y="28"/>
-<vertex x="297" y="28.1"/>
-<vertex x="297" y="210"/>
-<vertex x="0" y="210"/>
+<vertex x="297" y="200"/>
+<vertex x="0" y="200"/>
 </polygon>
 </signal>
