File: EAGLE/Analog/Analog_2.brd (EAGLE design)
At the start: 297 x 210 mm, 7 parts

Commit message: Я уже ничего не помню
Parts:
- moved 1 10.0 mm to (19.0, 75.5)
- moved E$1 10.0 mm to (19.0, 180.5)
- moved E$3 10.0 mm to (118.5, 75.5)
- moved E$4 10.0 mm to (118.5, 180.5)
- moved E$5 10.0 mm to (217.5, 75.5)
- moved E$6 10.0 mm to (217.5, 180.5)
- moved X1 10.0 mm to (284.0, 167.0)
Other:
- board size 297 x 210 mm -> 297 x 200 mm
