File: EAGLE/Analog/Analog_3.brd (EAGLE design)
At the start: 297 x 210 mm, 7 parts

Commit message: Я уже ничего не помню
Parts:
- moved 1 10.0 mm to (278.0, 75.5)
- moved E$1 10.0 mm to (278.0, 180.5)
- moved E$3 10.0 mm to (178.5, 75.5)
- moved E$4 10.0 mm to (178.5, 180.5)
- moved E$5 10.0 mm to (79.5, 75.5)
- moved E$6 10.0 mm to (79.5, 180.5)
- moved X1 10.0 mm to (13.0, 167.0)
Other:
- board size 297 x 210 mm -> 297 x 200 mm
